Commit message: update gazebo

File: catkin_ws/src/limo_ros/limo_description/urdf/limo_four_diff.xacro (robot description, xacro)
@@ -21,6 +21,21 @@
     <origin xyz="0.0 0.0 0.15" rpy="0 0 0"/>
   </joint>
+<!-- Base link -->
+    <link name="base_link">
+        <visual>
+            <origin xyz="0 0 -0.07" rpy="0 0 1.57" />
+            <geometry>
+                <box size="${base_x_size} ${base_y_size} ${base_z_size}"/>
+            </geometry>
+        </visual>
+        <collision>
+            <origin xyz="0 0 -0.07" rpy="0 0 1.57" />
+            <geometry>
+                <box size="${base_x_size} ${base_y_size} ${base_z_size}"/>
+            </geometry>
+        </collision>
+    </link>
     <!-- Base link -->
-    <link name="base_link">
+    <!-- <link name="base_link">
         <visual>
             <origin xyz="0 0 -0.15" rpy="0 0 1.57" />
@@ -29,12 +44,12 @@
             </geometry>
         </visual>
-        <collision>
+        <collision> -->
             <!--origin xyz="0 0 -0.15" rpy="0 0 1.57" /-->
-            <origin xyz="0 0 0" rpy="0 0 0" />
+            <!-- <origin xyz="0 0 0" rpy="0 0 0" />
           <geometry>
               <box size="${base_x_size} ${base_y_size} ${base_z_size}"/>
           </geometry>
         </collision>
-    </link>
+    </link> -->
     <link name="inertial_link">
         <inertial>

File: catkin_ws/src/limo_ros/limo_description/urdf/limo_xacro.xacro (robot description, xacro)
@@ -1,6 +1,5 @@
 git push origin main
 <?xml version="1.0"?>
-<robot name="limo_xacro" xmlns:xacro="http://ros.org/wiki/xacro">
-    <xacro:macro name="limo_wheel" params="parent_prefix wheel_prefix reflect *joint_pose">
+<xacro:macro name="limo_wheel" params="parent_prefix wheel_prefix reflect *joint_pose">
         <link name="${wheel_prefix}_wheel_link">
             <inertial>
@@ -10,14 +9,14 @@
             </inertial>
             <visual>
-                <origin xyz="0 0 0" rpy="0 0 0" />
+                <origin xyz="0 0 0" rpy="0 1.57 1.57" />
                 <geometry>
-                    <mesh filename="package://limo_description/meshes/limo_wheel.dae" />
+                    <cylinder length="${wheel_length}" radius="${wheel_radius}" />
                 </geometry>
             </visual>
             <collision>
-              <origin xyz="0 ${wheel_length/2} 0" rpy="1.57 0 0" />
-              <geometry>
-                  <cylinder length="${wheel_length}" radius="${wheel_radius}" />
-              </geometry>
+                <origin xyz="0 ${wheel_length/2} 0" rpy="0 1.57 1.57" />
+                <geometry>
+                    <cylinder length="${wheel_length}" radius="${wheel_radius}" />
+                </geometry>
             </collision>
         </link>

Commit message: UPDATE

File: catkin_ws/src/limo_ros/limo_description/urdf/limo_four_diff.xacro (robot description, xacro)
@@ -21,21 +21,6 @@
     <origin xyz="0.0 0.0 0.15" rpy="0 0 0"/>
   </joint>
-<!-- Base link -->
+    <!-- Base link -->
     <link name="base_link">
-        <visual>
-            <origin xyz="0 0 -0.07" rpy="0 0 1.57" />
-            <geometry>
-                <box size="${base_x_size} ${base_y_size} ${base_z_size}"/>
-            </geometry>
-        </visual>
-        <collision>
-            <origin xyz="0 0 -0.07" rpy="0 0 1.57" />
-            <geometry>
-                <box size="${base_x_size} ${base_y_size} ${base_z_size}"/>
-            </geometry>
-        </collision>
-    </link>
-    <!-- Base link -->
-    <!-- <link name="base_link">
         <visual>
             <origin xyz="0 0 -0.15" rpy="0 0 1.57" />
@@ -44,12 +29,12 @@
             </geometry>
         </visual>
-        <collision> -->
+        <collision>
             <!--origin xyz="0 0 -0.15" rpy="0 0 1.57" /-->
-            <!-- <origin xyz="0 0 0" rpy="0 0 0" />
+            <origin xyz="0 0 0" rpy="0 0 0" />
           <geometry>
               <box size="${base_x_size} ${base_y_size} ${base_z_size}"/>
           </geometry>
         </collision>
-    </link> -->
+    </link>
     <link name="inertial_link">
         <inertial>

File: catkin_ws/src/limo_ros/limo_description/urdf/limo_xacro.xacro (robot description, xacro)
@@ -1,5 +1,5 @@
-git push origin main
 <?xml version="1.0"?>
-<xacro:macro name="limo_wheel" params="parent_prefix wheel_prefix reflect *joint_pose">
+<robot name="limo_xacro" xmlns:xacro="http://ros.org/wiki/xacro">
+    <xacro:macro name="limo_wheel" params="parent_prefix wheel_prefix reflect *joint_pose">
         <link name="${wheel_prefix}_wheel_link">
             <inertial>
@@ -9,14 +9,14 @@
             </inertial>
             <visual>
-                <origin xyz="0 0 0" rpy="0 1.57 1.57" />
+                <origin xyz="0 0 0" rpy="0 0 0" />
                 <geometry>
-                    <cylinder length="${wheel_length}" radius="${wheel_radius}" />
+                    <mesh filename="package://limo_description/meshes/limo_wheel.dae" />
                 </geometry>
             </visual>
             <collision>
-                <origin xyz="0 ${wheel_length/2} 0" rpy="0 1.57 1.57" />
-                <geometry>
-                    <cylinder length="${wheel_length}" radius="${wheel_radius}" />
-                </geometry>
+              <origin xyz="0 ${wheel_length/2} 0" rpy="1.57 0 0" />
+              <geometry>
+                  <cylinder length="${wheel_length}" radius="${wheel_radius}" />
+              </geometry>
             </collision>
         </link>

Commit message: Add new thumbnail image for Lamp Post model in TurtleBot3 Autorace 2020

File: catkin_ws/src/limo_ros/limo_description/urdf/limo_four_diff.xacro (robot description, xacro)
@@ -24,15 +24,14 @@
     <link name="base_link">
         <visual>
-            <origin xyz="0 0 -0.15" rpy="0 0 1.57" />
+            <origin xyz="0 0 -0.07" rpy="0 0 1.57" />
             <geometry>
-                <mesh filename="package://limo_description/meshes/limo_base.dae" scale="1 1 1"/>
+                <box size="${base_x_size} ${base_y_size} ${base_z_size}"/>
             </geometry>
         </visual>
         <collision>
-            <!--origin xyz="0 0 -0.15" rpy="0 0 1.57" /-->
-            <origin xyz="0 0 0" rpy="0 0 0" />
-          <geometry>
-              <box size="${base_x_size} ${base_y_size} ${base_z_size}"/>
-          </geometry>
+            <origin xyz="0 0 -0.07" rpy="0 0 1.57" />
+            <geometry>
+                <box size="${base_x_size} ${base_y_size} ${base_z_size}"/>
+            </geometry>
         </collision>
     </link>

File: catkin_ws/src/limo_ros/limo_description/urdf/limo_xacro.xacro (robot description, xacro)
@@ -2,23 +2,23 @@
 <robot name="limo_xacro" xmlns:xacro="http://ros.org/wiki/xacro">
     <xacro:macro name="limo_wheel" params="parent_prefix wheel_prefix reflect *joint_pose">
-        <link name="${wheel_prefix}_wheel_link">
-            <inertial>
-                <origin xyz="0 0 0" />
-                <mass value="0.5" />
-                <inertia ixx="0.01055" ixy="0" ixz="0" iyy="0.00075" iyz="0" izz="0.01055" />
-            </inertial>
-            <visual>
-                <origin xyz="0 0 0" rpy="0 0 0" />
-                <geometry>
-                    <mesh filename="package://limo_description/meshes/limo_wheel.dae" />
-                </geometry>
-            </visual>
-            <collision>
-              <origin xyz="0 ${wheel_length/2} 0" rpy="1.57 0 0" />
-              <geometry>
-                  <cylinder length="${wheel_length}" radius="${wheel_radius}" />
-              </geometry>
-            </collision>
-        </link>
+            <link name="${wheel_prefix}_wheel_link">
+                <inertial>
+                    <origin xyz="0 0 0" />
+                    <mass value="0.5" />
+                    <inertia ixx="0.01055" ixy="0" ixz="0" iyy="0.00075" iyz="0" izz="0.01055" />
+                </inertial>
+                <visual>
+                    <origin xyz="0 0 0" rpy="0 1.57 1.57" />
+                    <geometry>
+                        <cylinder length="${wheel_length}" radius="${wheel_radius}" />
+                    </geometry>
+                </visual>
+                <collision>
+                    <origin xyz="0 ${wheel_length/2} 0" rpy="0 1.57 1.57" />
+                    <geometry>
+                        <cylinder length="${wheel_length}" radius="${wheel_radius}" />
+                    </geometry>
+                </collision>
+            </link>
         <joint name="${wheel_prefix}_wheel" type="continuous">
             <parent link="${parent_prefix}"/>
