Commit message: delete namespace limo

File: catkin_ws/src/abot/abot_description/urdf/robot.urdf.xacro (robot description, xacro)
@@ -148,5 +148,5 @@
     <child link="imu_link"/>
     <!--<origin xyz="-0.032 0 0.068" rpy="0 0 0"/>-->
-    <origin xyz="0 0 0" rpy="0 0 0"/>-->
+    <origin xyz="0 0 0" rpy="0 0 0"/>
   </joint>
   <link name="imu_link"/>

File: catkin_ws/src/limo_ros/limo_description/urdf/limo_four_diff_no_namespace.xacro (robot description, xacro)
@@ -1,7 +1,6 @@
 <?xml version="1.0"?>
 <robot name="limo_four_diff" xmlns:xacro="http://ros.org/wiki/xacro">
-    <xacro:arg name="robot_namespace" default="" />
     <xacro:include filename="$(find limo_description)/urdf/limo_xacro.xacro" />
-    <xacro:include filename="$(find limo_description)/urdf/limo_four_diff.gazebo" />
+    <xacro:include filename="$(find limo_description)/urdf/limo_four_diff_no_namespace.gazebo" />
     <!-- Variables -->
     <xacro:property name="M_PI" value="3.14159"/>
